File: kicad/roz-power-board.kicad_pcb (KiCad board)
At the start: 2 copper layers, 80 x 42 mm, 85 parts, among them CON1 USB-MICRO-B, J1 Jumper_Switch, J2 Jumper_Switch, J3 Jumper_Switch, J4 Jumper_Switch, J5 Jumper_Switch, J6 Jumper_Switch, P1 Wall Power, P10 GPIO_A5, P11 GPIO_A6, P12 GPIO_A7, P13 BIOLOID_BUS_1, P14 LED, P15 Bus Switch, P16 BIOLOID_BUS_2, P17 BIOLOID_BUS_3, P18 BIOLOID_BUS_4, P19 BIOLOID_BUS_5, P2 Battery, P20 BIOLOID_BUS_6, P21 rPi, P25 VBAT, P26 BUS, P3 BATT_BALANCE, P4 ALT_3.3, P5 UART_1, P6 I2C_2, P7 SPI_2, P8 5V Regulator, P9 GPIO_A4, Q1 BS-170, Q2 STD30PF03LT4, Q3 STD30PF03LT4, SW2 PowerSwitch, SW3 RESET_SW, SW4 BOOT_SW, U1 LM3480-3.3, U2 LTC4412, U3 STM32F401xD_UFQFPN48, X1 32.768kHz, X2 8MHz

Commit message: rev 0.2 of the power board
Parts:
- added P23: USR_SW, MicroPython-Parts-new:SIL_2_050, F.Cu at (158.7, 122.9)
- added P_JUMP: P_JUMP, Socket_Strips:Socket_Strip_Straight_1x02, F.Cu at (124.0, 113.1)
- U1: value LM3480-3.3 -> AP7333
- moved P13 25.4 mm to (131.4, 105.5)
- moved P20 25.0 mm to (156.4, 105.5)
- moved P16 15.3 mm to (136.4, 105.5)
- moved P19 9.91 mm to (146.4, 105.5)
- moved P18 9.83 mm to (151.4, 105.5)
- moved P17 5.25 mm to (141.4, 105.5)
- moved C1 5.05 mm to (138.1, 133.5)
- moved C2 5.00 mm to (133.0, 133.5)
- moved C14 2.05 mm to (115.7, 115.2)
- moved P3 1.00 mm to (164.6, 139.3)
- moved P8 0.25 mm to (155.8, 140.2)
- moved C3 0.15 mm to (102.5, 128.2)
- moved U1 0.05 mm to (135.5, 133.7)
Connections:
- Q2 pad 2: +F_POWER -> +12V
- Q2 pad 3: +12V -> +F_POWER
- R24 pad 2: Net-(R24-Pad2) -> BOOT0
- SW4 pad 1: Net-(R24-Pad2) -> BOOT0
- U1 pad 1: +3V3 -> +5V
- U1 pad 2: +5V -> +3V3
- U3 pad 44: Net-(R24-Pad2) -> BOOT0
- U3 pad 45: Net-(U3-Pad45) -> BOOT0
Routing:
- net Net-(P23-Pad2): track 0.00 -> 15.6 mm, vias 0 -> 1
- net +5V: track 108.1 -> 96.8 mm, vias 3 -> 1
- net +3V3: track 193.7 -> 202.3 mm, vias 14 -> 12
- net Net-(P22-Pad2): track 19.8 -> 27.2 mm
- net BOOT0: track 0.00 -> 7.15 mm
- net Net-(R24-Pad2): track 5.59 -> 0.00 mm
- net +F_POWER: track 21.5 -> 16.5 mm
- net +12V: track 73.1 -> 69.2 mm
- net GND: track 67.1 -> 69.0 mm
- net VBAT: track 19.2 -> 19.6 mm, vias 0 -> 1
Other:
- board text added: "+12"
- board text added: "Jon & Dave Hylands Bioloid Power Board v. 0.2 powered by MicroPython"
- board text removed: "Jon & Dave Hylands Bioloid Power Board powered by MicroPython"
